Commit message: urdf 100%. now straight to bridge and api

File: slrc_tron_sim/urdf/lightcycle.urdf (robot description, URDF)
Before this commit: robot slrc_lightcycle, 11 links, 10 joints
Links:
- removed link front_left_wheel
- removed link front_right_wheel
- removed link rear_left_wheel
- removed link rear_right_wheel
- added link left_wheel_link, mass 0.10; collision cylinder length=0.01 radius=0.02
- added link right_wheel_link, mass 0.10; collision cylinder length=0.01 radius=0.02
- link base_link: mass 18.0 -> 4.0; geometry collision box size=0.18 0.06 0.081; visual mesh filename=package://slrc_tron_sim/meshes/lightcycle.STL scale=0.001 0.001 0.0015
- link led_link: geometry visual cylinder length=0.015 radius=0.005; visual sphere radius=0.008
Joints:
- removed joint front_left_wheel_joint
- removed joint front_right_wheel_joint
- removed joint rear_left_wheel_joint
- removed joint rear_right_wheel_joint
- added joint left_wheel_joint: type continuous, parent base_link, child left_wheel_link, origin xyz=0.0 0.035 0.021 rpy=1.5708 0 0, axis 0 1 0
- added joint right_wheel_joint: type continuous, parent base_link, child right_wheel_link, origin xyz=0 -0.035 0.021 rpy=1.5708 0 0, axis 0 1 0
- joint led_fixed: origin xyz=0 0 0 rpy=0 0 0 -> xyz=-0.05 0 0.058 rpy=0 0 0

Commit message: got the api and bridge up as propsed architecture but robot stop responding after the initial command

File: slrc_tron_sim/urdf/lightcycle.urdf (robot description, URDF)
Before this commit: robot slrc_lightcycle, 9 links, 8 joints
Links:
- link left_wheel_link: mass 0.10 -> 0.2; geometry collision cylinder length=0.02 radius=0.033
- link right_wheel_link: mass 0.10 -> 0.2; geometry collision cylinder length=0.02 radius=0.033
Joints:
- joint left_wheel_joint: origin xyz=0.0 0.035 0.021 rpy=1.5708 0 0 -> xyz=0.0 0.035 0.033 rpy=0 0 0
- joint right_wheel_joint: origin xyz=0 -0.035 0.021 rpy=1.5708 0 0 -> xyz=0 -0.035 0.033 rpy=0 0 0

Commit message: Issue was the ground lines having significantly tall collision meshes. now working as expected

File: slrc_tron_sim/urdf/lightcycle.urdf (robot description, URDF)
Before this commit: robot slrc_lightcycle, 9 links, 8 joints
Joints:
- joint left_wheel_joint: origin xyz=0.0 0.035 0.033 rpy=0 0 0 -> xyz=0.0 0.05 0.033 rpy=0 0 0
- joint right_wheel_joint: origin xyz=0 -0.035 0.033 rpy=0 0 0 -> xyz=0 -0.05 0.033 rpy=0 0 0
