Commit message: cameras working. issue was forgoting to add the senor and physics plugins to the world all alone. Right now rendering using creating virtual frame buffer using xvfb and forwarding it using a vnc server. Will change that to previous method but might need this for the final server deployment

File: src/slrc_tron_sim/urdf/hostile_agent.urdf (robot description, URDF)
Before this commit: robot hostile_agent, 5 links, 4 joints
Links:
- added link cam_floor_link
Joints:
- added joint cam_floor_fixed: type fixed, parent base_link, child cam_floor_link, origin xyz=0.15 0.0 0.18 rpy=0 1.5708 0
