Commit message: cleaned up the repo

File: src/slrc_tron_sim/urdf/ares.urdf (robot description, URDF)
Before this commit: robot ares, 9 links, 8 joints
Joints:
- joint cam_front_left_fixed: origin xyz=0.45 0.10 0.45 rpy=0 0 0 -> xyz=0.45 0.10 0.45 rpy=0 0 0.7854
- joint cam_front_right_fixed: origin xyz=0.45 -0.10 0.45 rpy=0 0 0 -> xyz=0.45 -0.10 0.45 rpy=0 0 -0.7854

Commit message: added forgotten plugin to the urdf. need to test

File: src/slrc_tron_sim/urdf/ares.urdf (robot description, URDF)
Before this commit: robot ares, 9 links, 8 joints
Joints:
- joint imu_fixed: origin xyz=0 0 0.35 rpy=0 0 0 -> xyz=0 0 0.05 rpy=0 0 0

Commit message: led feature added

File: src/slrc_tron_sim/urdf/ares.urdf (robot description, URDF)
Before this commit: robot ares, 9 links, 8 joints
Links:
- added link led_base_link; visual cylinder length=0.015 radius=0.005
- link led_link: geometry visual sphere radius=0.008
Joints:
- removed joint led_fixed
- added joint led_base_fixed: type fixed, parent base_link, child led_base_link, origin xyz=-0.05 0 0.058 rpy=0 0 0
- added joint led_dome_fixed: type fixed, parent led_base_link, child led_link, origin xyz=0 0 0.015 rpy=0 0 0

File: src/slrc_tron_sim/urdf/hostile_agent.urdf (robot description, URDF)
Before this commit: robot hostile_agent, 6 links, 5 joints
Links:
- removed link base_footprint
- added link hostile_base_footprint
Joints:
- joint base_footprint_to_base: parent base_footprint -> hostile_base_footprint
